File: kicad/287-booster.kicad_sch (KiCad schematic)
At the start: 4 parts, among them J1 Conn_01x02_Female, U1 80287, U2 Socket

Commit message: Update to KiCad 9
Changed lines of the file:
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@@
 (kicad_sch
-	(version 20231120)
+	(version 20250114)
 	(generator "eeschema")
-	(generator_version "8.0")
+	(generator_version "9.0")
 	(paper "A4")
 	(title_block
@@
 	(label "~{NPS1}"
 		(at 185.42 113.03 0)
-		(fields_autoplaced yes)
 		(effects
 			(font
@@
 	(label "D2"
 		(at 134.62 146.05 0)
-		(fields_autoplaced yes)
 		(effects
 			(font
@@
 	(label "~{INTA}"
 		(at 144.78 102.87 0)
-		(fields_autoplaced yes)
 		(effects
 			(font
@@
 	(label "~{PEACK}"
 		(at 130.81 107.95 0)
-		(fields_autoplaced yes)
 		(effects
 			(font
@@
 	(label "CMD0"
 		(at 132.08 125.73 0)
-		(fields_autoplaced yes)
 		(effects
 			(font
@@
 	(label "~{READY}"
 		(at 130.81 97.79 0)
-		(fields_autoplaced yes)
 		(effects
 			(font
@@
 	(label "D12"
 		(at 144.78 115.57 0)
-		(fields_autoplaced yes)
 		(effects
 			(font
@@
 	(label "D4"
 		(at 144.78 143.51 0)
-		(fields_autoplaced yes)
 		(effects
 			(font
@@
 	(label "D1"
 		(at 187.96 143.51 0)
-		(fields_autoplaced yes)
 		(effects
 			(font
@@
 	(label "~{S0}"
 		(at 144.78 100.33 0)
-		(fields_autoplaced yes)
 		(effects
 			(font
@@
 	(label "D4"
 		(at 91.44 143.51 0)
-		(fields_autoplaced yes)
 		(effects
 			(font
@@
 	(label "~{PEACK}"
 		(at 184.15 107.95 0)
-		(fields_autoplaced yes)
 		(effects
 			(font
@@
 	(label "CLK"
 		(at 133.35 118.11 0)
-		(fields_autoplaced yes)
 		(effects
 			(font
@@
 	(label "D13"
 		(at 91.44 113.03 0)
-		(fields_autoplaced yes)
 		(effects
 			(font
@@
 	(label "PEREQ"
 		(at 184.15 138.43 0)
-		(fields_autoplaced yes)
 		(effects
 			(font
@@
 	(label "D2"
 		(at 187.96 146.05 0)
-		(fields_autoplaced yes)
 		(effects
 			(font
@@
 	(label "NC13"
 		(at 144.78 128.27 0)
-		(fields_autoplaced yes)
 		(effects
 			(font
@@
 	(label "D5"
 		(at 91.44 140.97 0)
-		(fields_autoplaced yes)
 		(effects
 			(font
@@
 	(label "~{BUSY}"
 		(at 132.08 135.89 0)
-		(fields_autoplaced yes)
 		(effects
 			(font
@@
 	(label "HLDA"
 		(at 132.08 102.87 0)
-		(fields_autoplaced yes)
 		(effects
 			(font
@@
 	(label "D8"
 		(at 144.78 133.35 0)
-		(fields_autoplaced yes)
 		(effects
 			(font
@@
 	(label "HLDA"
 		(at 185.42 102.87 0)
-		(fields_autoplaced yes)
 		(effects
 			(font
@@
 	(label "D3"
 		(at 91.44 146.05 0)
-		(fields_autoplaced yes)
 		(effects
 			(font
@@
 	(label "D7"
 		(at 91.44 135.89 0)
-		(fields_autoplaced yes)
 		(effects
 			(font
@@
 	(label "~{S1}"
 		(at 91.44 97.79 0)
-		(fields_autoplaced yes)
 		(effects
 			(font
@@
 	(label "D13"
 		(at 144.78 113.03 0)
-		(fields_autoplaced yes)
 		(effects
 			(font
@@
 	(label "D14"
 		(at 91.44 110.49 0)
-		(fields_autoplaced yes)
 		(effects
 			(font
@@
 	(label "D5"
 		(at 144.78 140.97 0)
-		(fields_autoplaced yes)
 		(effects
 			(font
@@
 	(label "RESET"
 		(at 184.15 110.49 0)
-		(fields_autoplaced yes)
 		(effects
 			(font
@@
 	(label "D8"
 		(at 91.44 133.35 0)
-		(fields_autoplaced yes)
 		(effects
 			(font
@@
 	(label "~{S1}"
 		(at 144.78 97.79 0)
-		(fields_autoplaced yes)
 		(effects
 			(font
@@
 	(label "D0"
 		(at 134.62 140.97 0)
-		(fields_autoplaced yes)
 		(effects
 			(font
@@
 	(label "D1"
 		(at 134.62 143.51 0)
-		(fields_autoplaced yes)
 		(effects
 			(font
@@
 	(label "~{BUSY}"
 		(at 185.42 135.89 0)
-		(fields_autoplaced yes)
 		(effects
 			(font
@@
 	(label "D6"
 		(at 144.78 138.43 0)
-		(fields_autoplaced yes)
 		(effects
 			(font
@@
 	(label "D14"
 		(at 144.78 110.49 0)
-		(fields_autoplaced yes)
 		(effects
 			(font
@@
 	(label "D15"
 		(at 144.78 107.95 0)
-		(fields_autoplaced yes)
 		(effects
 			(font
@@
 	(label "~{NPRD}"
 		(at 185.42 130.81 0)
-		(fields_autoplaced yes)
 		(effects
 			(font
@@
 	(label "CLK286"
 		(at 182.88 105.41 0)
-		(fields_autoplaced yes)
 		(effects
 			(font
@@
 	(label "D6"
 		(at 91.44 138.43 0)
-		(fields_autoplaced yes)
 		(effects
 			(font
@@
 	(label "~{ERROR}"
 		(at 184.15 133.35 0)
-		(fields_autoplaced yes)
 		(effects
 			(font
@@
 	(label "CLK"
 		(at 186.69 118.11 0)
-		(fields_autoplaced yes)
 		(effects
 			(font
@@
 	(label "NPS2"
 		(at 185.42 115.57 0)
-		(fields_autoplaced yes)
 		(effects
 			(font
@@
 	(label "D0"
 		(at 187.96 140.97 0)
-		(fields_autoplaced yes)
 		(effects
 			(font
@@
 	(label "PEREQ"
 		(at 130.81 138.43 0)
-		(fields_autoplaced yes)
 		(effects
 			(font
@@
 	(label "~{INTA}"
 		(at 91.44 102.87 0)
-		(fields_autoplaced yes)
 		(effects
 			(font
@@
 	(label "NC4"
 		(at 91.44 105.41 0)
-		(fields_autoplaced yes)
 		(effects
 			(font
@@
 	(label "~{ERROR}"
 		(at 130.81 133.35 0)
-		(fields_autoplaced yes)
 		(effects
 			(font
@@
 	(label "D12"
 		(at 91.44 115.57 0)
-		(fields_autoplaced yes)
 		(effects
 			(font
@@
 	(label "CMD1"
 		(at 132.08 120.65 0)
-		(fields_autoplaced yes)
 		(effects
 			(font
@@
 	(label "D10"
 		(at 144.78 125.73 0)
-		(fields_autoplaced yes)
 		(effects
 			(font
@@
 	(label "CLK286"
 		(at 129.54 105.41 0)
-		(fields_autoplaced yes)
 		(effects
 			(font
@@
 	(label "~{NPWR}"
 		(at 132.08 128.27 0)
-		(fields_autoplaced yes)
 		(effects
 			(font
@@
 	(label "NPS2"
 		(at 132.08 115.57 0)
-		(fields_autoplaced yes)
 		(effects
 			(font
@@
 	(label "NC4"
 		(at 144.78 105.41 0)
-		(fields_autoplaced yes)
 		(effects
 			(font
@@
 	(label "~{S0}"
 		(at 91.44 100.33 0)
-		(fields_autoplaced yes)
 		(effects
 			(font
@@
 	(label "D15"
 		(at 91.44 107.95 0)
-		(fields_autoplaced yes)
 		(effects
 			(font
@@
 	(label "~{NPRD}"
 		(at 132.08 130.81 0)
-		(fields_autoplaced yes)
 		(effects
 			(font
@@
 	(label "~{NPS1}"
 		(at 132.08 113.03 0)
-		(fields_autoplaced yes)
 		(effects
 			(font
@@
 	(label "CMD1"
 		(at 185.42 120.65 0)
-		(fields_autoplaced yes)
 		(effects
 			(font
@@
 	(label "~{NPWR}"
 		(at 185.42 128.27 0)
-		(fields_autoplaced yes)
 		(effects
 			(font
@@
 	(label "D11"
 		(at 144.78 123.19 0)
-		(fields_autoplaced yes)
 		(effects
 			(font
@@
 	(label "D9"
 		(at 144.78 130.81 0)
-		(fields_autoplaced yes)
 		(effects
 			(font
@@
 	(label "CMD0"
 		(at 185.42 125.73 0)
-		(fields_autoplaced yes)
 		(effects
 			(font
@@
 	(label "D7"
 		(at 144.78 135.89 0)
-		(fields_autoplaced yes)
 		(effects
 			(font
@@
 	(label "D3"
 		(at 144.78 146.05 0)
-		(fields_autoplaced yes)
 		(effects
 			(font
@@
 	(label "RESET"
 		(at 130.81 110.49 0)
-		(fields_autoplaced yes)
 		(effects
 			(font
@@
 	(label "D11"
 		(at 91.44 123.19 0)
-		(fields_autoplaced yes)
 		(effects
 			(font
@@
 	(label "~{READY}"
 		(at 184.15 97.79 0)
-		(fields_autoplaced yes)
 		(effects
 			(font
@@
 	(label "NC13"
 		(at 91.44 128.27 0)
-		(fields_autoplaced yes)
 		(effects
 			(font
@@
 	(label "D10"
 		(at 91.44 125.73 0)
-		(fields_autoplaced yes)
 		(effects
 			(font
@@
 	(label "D9"
 		(at 91.44 130.81 0)
-		(fields_autoplaced yes)
 		(effects
 			(font
@@
 		)
 	)
+	(embedded_fonts no)
 )
