File: kicad/287-booster.kicad_pcb (KiCad board)
At the start: 2 copper layers, 24.9 x 51.6 mm, 5 parts, among them J1 Conn_01x02_Female, U1 80287, U2 Socket

Commit message: rotated text
Parts:
- turned REF** to -90 degrees
Changed lines of the file:
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@@
 			(psa4output no)
 			(plot_black_and_white yes)
-			(plotinvisibletext no)
 			(sketchpadsonfab no)
 			(plotpadnumbers no)
@@
 		(tags "Through hole pin header THT 1x02 2.54mm single row")
 		(property "Reference" "J1"
-			(at 0 4.826 270)
+			(at 0 4.826 0)
 			(layer "F.SilkS")
 			(effects
@@
 		(tags "THT DIP DIL PDIP 2.54mm 15.24mm 600mil Socket")
 		(property "Reference" "U1"
-			(at 7.62 0.762 90)
+			(at 7.62 0.762 0)
 			(layer "F.SilkS")
 			(effects
@@
 		)
 		(property "Value" "80287"
-			(at 7.62 24.129001 90)
+			(at 9.144 24.125 180)
 			(layer "F.SilkS")
 			(effects
@@
 	(footprint "Symbol:OSHW-Logo2_9.8x8mm_Copper"
 		(layer "F.Cu")
-		(at 150.876 99.06 90)
+		(at 150.876 99.06 -90)
 		(descr "Open Source Hardware Symbol")
 		(tags "Logo Symbol OSHW")
@@
 		)
 		(property "Datasheet" ""
-			(at 0 0 90)
+			(at 0 0 270)
 			(unlocked yes)
 			(layer "F.Fab")
@@
 		)
 		(property "Description" ""
-			(at 0 0 90)
+			(at 0 0 270)
 			(unlocked yes)
 			(layer "F.Fab")
@@
 		(fp_poly
 			(pts
+				(xy 2.887333 2.633528) (xy 2.94359 2.659117) (xy 2.987747 2.690124) (xy 3.020101 2.724795) (xy 3.042438 2.76952)
+				(xy 3.056546 2.830692) (xy 3.064211 2.914701) (xy 3.06722 3.02794) (xy 3.067538 3.102509) (xy 3.067538 3.39342)
+				(xy 3.017773 3.416095) (xy 2.978576 3.432667) (xy 2.959157 3.438769) (xy 2.955442 3.42061) (xy 2.952495 3.371648)
+				(xy 2.950691 3.300153) (xy 2.950308 3.243385) (xy 2.948661 3.161371) (xy 2.944222 3.096309) (xy 2.93774 3.056467)
+				(xy 2.93259 3.048) (xy 2.897977 3.056646) (xy 2.84364 3.078823) (xy 2.780722 3.108886) (xy 2.720368 3.141192)
+				(xy 2.673721 3.170098) (xy 2.651926 3.189961) (xy 2.651839 3.190175) (xy 2.653714 3.226935) (xy 2.670525 3.262026)
+				(xy 2.700039 3.290528) (xy 2.743116 3.300061) (xy 2.779932 3.29895) (xy 2.832074 3.298133) (xy 2.859444 3.310349)
+				(xy 2.875882 3.342624) (xy 2.877955 3.34871) (xy 2.885081 3.394739) (xy 2.866024 3.422687) (xy 2.816353 3.436007)
+				(xy 2.762697 3.43847) (xy 2.666142 3.42021) (xy 2.616159 3.394131) (xy 2.554429 3.332868) (xy 2.52169 3.25767)
+				(xy 2.518753 3.178211) (xy 2.546424 3.104167) (xy 2.588047 3.057769) (xy 2.629604 3.031793) (xy 2.694922 2.998907)
+				(xy 2.771038 2.965557) (xy 2.783726 2.960461) (xy 2.867333 2.923565) (xy 2.91553 2.891046) (xy 2.93103 2.858718)
+				(xy 2.91655 2.822394) (xy 2.891692 2.794) (xy 2.832939 2.759039) (xy 2.768293 2.756417) (xy 2.709008 2.783358)
+				(xy 2.666339 2.837088) (xy 2.660739 2.85095) (xy 2.628133 2.901936) (xy 2.58053 2.939787) (xy 2.520461 2.97085)
+				(xy 2.520461 2.882768) (xy 2.523997 2.828951) (xy 2.539156 2.786534) (xy 2.572768 2.741279) (xy 2.605035 2.70642)
+				(xy 2.655209 2.657062) (xy 2.694193 2.630547) (xy 2.736064 2.619911) (xy 2.78346 2.618154) (xy 2.887333 2.633528)
+			)
+			(stroke
+				(width 0.01)
+				(type solid)
+			)
+			(fill yes)
+			(layer "F.Mask")
+		)
+		(fp_poly
+			(pts
 				(xy -3.231114 2.584505) (xy -3.156461 2.621727) (xy -3.090569 2.690261) (xy -3.072423 2.715648)
 				(xy -3.052655 2.748866) (xy -3.039828 2.784945) (xy -3.03249 2.833098) (xy -3.029187 2.902536) (xy -3.028462 2.994206)
@@
 				(xy -3.626742 2.753555) (xy -3.616857 2.729668) (xy -3.603954 2.708764) (xy -3.598421 2.700898)
 				(xy -3.525031 2.626595) (xy -3.43224 2.584467) (xy -3.324904 2.572722) (xy -3.231114 2.584505)
-			)
-			(stroke
-				(width 0.01)
-				(type solid)
-			)
-			(fill yes)
-			(layer "F.Mask")
-		)
-		(fp_poly
-			(pts
-				(xy 2.887333 2.633528) (xy 2.94359 2.659117) (xy 2.987747 2.690124) (xy 3.020101 2.724795) (xy 3.042438 2.76952)
-				(xy 3.056546 2.830692) (xy 3.064211 2.914701) (xy 3.06722 3.02794) (xy 3.067538 3.102509) (xy 3.067538 3.39342)
-				(xy 3.017773 3.416095) (xy 2.978576 3.432667) (xy 2.959157 3.438769) (xy 2.955442 3.42061) (xy 2.952495 3.371648)
-				(xy 2.950691 3.300153) (xy 2.950308 3.243385) (xy 2.948661 3.161371) (xy 2.944222 3.096309) (xy 2.93774 3.056467)
-				(xy 2.93259 3.048) (xy 2.897977 3.056646) (xy 2.84364 3.078823) (xy 2.780722 3.108886) (xy 2.720368 3.141192)
-				(xy 2.673721 3.170098) (xy 2.651926 3.189961) (xy 2.651839 3.190175) (xy 2.653714 3.226935) (xy 2.670525 3.262026)
-				(xy 2.700039 3.290528) (xy 2.743116 3.300061) (xy 2.779932 3.29895) (xy 2.832074 3.298133) (xy 2.859444 3.310349)
-				(xy 2.875882 3.342624) (xy 2.877955 3.34871) (xy 2.885081 3.394739) (xy 2.866024 3.422687) (xy 2.816353 3.436007)
-				(xy 2.762697 3.43847) (xy 2.666142 3.42021) (xy 2.616159 3.394131) (xy 2.554429 3.332868) (xy 2.52169 3.25767)
-				(xy 2.518753 3.178211) (xy 2.546424 3.104167) (xy 2.588047 3.057769) (xy 2.629604 3.031793) (xy 2.694922 2.998907)
-				(xy 2.771038 2.965557) (xy 2.783726 2.960461) (xy 2.867333 2.923565) (xy 2.91553 2.891046) (xy 2.93103 2.858718)
-				(xy 2.91655 2.822394) (xy 2.891692 2.794) (xy 2.832939 2.759039) (xy 2.768293 2.756417) (xy 2.709008 2.783358)
-				(xy 2.666339 2.837088) (xy 2.660739 2.85095) (xy 2.628133 2.901936) (xy 2.58053 2.939787) (xy 2.520461 2.97085)
-				(xy 2.520461 2.882768) (xy 2.523997 2.828951) (xy 2.539156 2.786534) (xy 2.572768 2.741279) (xy 2.605035 2.70642)
-				(xy 2.655209 2.657062) (xy 2.694193 2.630547) (xy 2.736064 2.619911) (xy 2.78346 2.618154) (xy 2.887333 2.633528)
 			)
 			(stroke
@@
 		(tags "Resistor Axial_DIN0207 series Axial Horizontal pin pitch 7.62mm 0.25W = 1/4W length 6.3mm diameter 2.5mm")
 		(property "Reference" "R1"
-			(at -2.286 0 270)
+			(at -2.54 0 0)
 			(layer "F.SilkS")
 			(effects
@@
 		)
 		(property "Value" "10K"
-			(at 3.81 -0.0675 90)
+			(at 3.81 0 90)
 			(layer "F.SilkS")
 			(effects
@@
 		)
 		(fp_text user "${REFERENCE}"
-			(at -2.54 0 180)
+			(at -2.54 0 0)
 			(layer "F.Fab")
 			(effects
@@
 	)
 	(gr_text "287 Booster by i440bx & Necroware"
-		(at 163.068 108.712 90)
+		(at 163.195 77.724 270)
 		(layer "F.Mask")
 		(effects
@@
 	)
 	(gr_text "on: clk/1\noff: clk/n"
-		(at 163.068 74.676 90)
+		(at 163.195 66.802 270)
 		(layer "F.SilkS")
 		(effects
@@
 	)
 	(segment
-		(start 154.432 64.77)
+		(start 156.972 62.23)
+		(end 151.9595 62.23)
+		(width 0.25)
+		(layer "B.Cu")
+		(net 3)
+	)
+	(segment
+		(start 151.9595 62.23)
 		(end 149.4195 64.77)
 		(width 0.25)
 		(layer "B.Cu")
-		(net 3)
-	)
-	(segment
-		(start 156.972 62.23)
-		(end 154.432 64.77)
-		(width 0.25)
-		(layer "B.Cu")
